File: Chua.brd (EAGLE design)
At the start: 37.8 x 44.4 mm, 17 parts, among them IC1 LT1001, J1 ZYX, J2 E-,E+

Commit message: 1.1
Fixed mistake R8 should be a trimmer instead of a resistor.
Parts:
- R8: value 1530 -> (none); device resistor:0204/7 -> resistor:RTRIM3296Y
- moved R8 7.73 mm to (22.9, 36.8), turned to 180 degrees
Connections:
- net N$6: now also R8.1
- net N$7: now also R8.3; no longer R8.1
Routing:
- net N$7: track 17.8 -> 19.0 mm
- net N$6: track 58.5 -> 57.8 mm
Changed lines of the file:
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@@
 <layers>
 <layer number="1" name="Top" color="4" fill="1" visible="yes" active="yes"/>
+<layer number="2" name="Route2" color="1" fill="3" visible="no" active="no"/>
+<layer number="3" name="Route3" color="4" fill="3" visible="no" active="no"/>
+<layer number="4" name="Route4" color="1" fill="4" visible="no" active="no"/>
+<layer number="5" name="Route5" color="4" fill="4" visible="no" active="no"/>
+<layer number="6" name="Route6" color="1" fill="8" visible="no" active="no"/>
+<layer number="7" name="Route7" color="4" fill="8" visible="no" active="no"/>
+<layer number="8" name="Route8" color="1" fill="2" visible="no" active="no"/>
+<layer number="9" name="Route9" color="4" fill="2" visible="no" active="no"/>
+<layer number="10" name="Route10" color="1" fill="7" visible="no" active="no"/>
+<layer number="11" name="Route11" color="4" fill="7" visible="no" active="no"/>
+<layer number="12" name="Route12" color="1" fill="5" visible="no" active="no"/>
+<layer number="13" name="Route13" color="4" fill="5" visible="no" active="no"/>
+<layer number="14" name="Route14" color="1" fill="6" visible="no" active="no"/>
+<layer number="15" name="Route15" color="4" fill="6" visible="no" active="no"/>
 <layer number="16" name="Bottom" color="1" fill="1" visible="yes" active="yes"/>
 <layer number="17" name="Pads" color="2" fill="1" visible="yes" active="yes"/>
@@
 <element name="R6" library="resistor" package="0204/7" value="47K" x="16.51" y="12.7"/>
 <element name="R7" library="resistor" package="0204/7" value="3.3K" x="16.51" y="5.08" rot="R180"/>
-<element name="R8" library="resistor" package="0204/7" value="1530" x="21.59" y="29.21" rot="R270"/>
 <element name="R9" library="resistor" package="0204/7" value="10" x="12.7" y="24.13" rot="R90"/>
 <element name="D1" library="diode" package="DO35-7" value="1N4148DO35-7" x="16.51" y="8.89" rot="R180"/>
@@
 <element name="J1" library="con-amp" package="10X03MTA" value="ZYX" x="15.24" y="39.37" rot="R180"/>
 <element name="J2" library="con-amp" package="10X02MTA" value="E-,E+" x="29.21" y="39.37" rot="R180"/>
+<element name="R8" library="resistor" package="RTRIM3296Y" value="" x="22.86" y="36.83" rot="R180"/>
 </elements>
 <signals>
@@
 <contactref element="D2" pad="A"/>
 <contactref element="R2" pad="2"/>
-<contactref element="R8" pad="2"/>
 <contactref element="IC1" pad="3"/>
 <contactref element="C1" pad="1"/>
@@
 <wire x1="20.32" y1="8.89" x2="24.13" y2="8.89" width="0.4064" layer="16"/>
 <wire x1="24.13" y1="8.89" x2="24.13" y2="11.43" width="0.4064" layer="16"/>
-<wire x1="19.05" y1="21.59" x2="21.59" y2="21.59" width="0.4064" layer="16"/>
-<wire x1="21.59" y1="21.59" x2="21.59" y2="24.13" width="0.4064" layer="16"/>
-<wire x1="21.59" y1="24.13" x2="21.59" y2="25.4" width="0.4064" layer="16"/>
+<contactref element="R8" pad="1"/>
+<contactref element="R8" pad="2"/>
 <wire x1="31.75" y1="21.59" x2="29.21" y2="24.13" width="0.4064" layer="16"/>
 <wire x1="29.21" y1="24.13" x2="21.59" y2="24.13" width="0.4064" layer="16"/>
-<wire x1="21.59" y1="25.4" x2="21.59" y2="29.21" width="0.4064" layer="16"/>
-<wire x1="21.59" y1="29.21" x2="24.13" y2="31.75" width="0.4064" layer="16"/>
-<wire x1="24.13" y1="31.75" x2="24.13" y2="35.56" width="0.4064" layer="16"/>
-<wire x1="24.13" y1="35.56" x2="20.32" y2="39.37" width="0.4064" layer="16"/>
-<wire x1="20.32" y1="39.37" x2="17.78" y2="39.37" width="0.4064" layer="16"/>
+<wire x1="19.05" y1="21.59" x2="21.59" y2="24.13" width="0.4064" layer="16"/>
+<wire x1="21.59" y1="24.13" x2="21.59" y2="30.48" width="0.4064" layer="16"/>
+<wire x1="21.59" y1="30.48" x2="24.13" y2="33.02" width="0.4064" layer="16"/>
+<wire x1="24.13" y1="33.02" x2="24.13" y2="36.83" width="0.4064" layer="16"/>
+<wire x1="24.13" y1="36.83" x2="21.59" y2="39.37" width="0.4064" layer="16"/>
+<wire x1="21.59" y1="39.37" x2="17.78" y2="39.37" width="0.4064" layer="16"/>
 </signal>
 <signal name="N$2">
@@
 <signal name="N$7">
 <contactref element="C2" pad="1"/>
-<contactref element="R8" pad="1"/>
 <contactref element="L1" pad="2"/>
 <contactref element="J1" pad="2"/>
 <wire x1="15.24" y1="33.02" x2="15.24" y2="39.37" width="0.4064" layer="16"/>
 <wire x1="17.78" y1="33.02" x2="19.05" y2="33.02" width="0.4064" layer="16"/>
-<wire x1="19.05" y1="33.02" x2="21.59" y2="33.02" width="0.4064" layer="16"/>
 <wire x1="19.05" y1="27.94" x2="19.05" y2="33.02" width="0.4064" layer="16"/>
 <wire x1="17.78" y1="33.02" x2="15.24" y2="33.02" width="0.4064" layer="16"/>
+<contactref element="R8" pad="3"/>
+<wire x1="19.05" y1="33.02" x2="21.59" y2="33.02" width="0.4064" layer="16"/>
+<wire x1="21.59" y1="33.02" x2="21.59" y2="34.29" width="0.4064" layer="16"/>
 </signal>
 <signal name="N$8">
