File: Chua.sch (EAGLE design)
At the start: 17 parts, among them IC1 LT1001, J1 ZYX, J2 E-,E+

Commit message: 1.1
Fixed mistake R8 should be a trimmer instead of a resistor.
Parts:
- R8: value 1530 -> (none); device resistor:R-US_0204/7 -> resistor:R-TRIMM3296Y
Connections:
- net N$6: now also R8.E, R8.S; no longer R8.2
- net N$7: now also R8.A; no longer R8.1
Changed lines of the file:
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@@
 <layers>
 <layer number="1" name="Top" color="4" fill="1" visible="no" active="no"/>
+<layer number="2" name="Route2" color="1" fill="3" visible="no" active="no"/>
+<layer number="3" name="Route3" color="4" fill="3" visible="no" active="no"/>
+<layer number="4" name="Route4" color="1" fill="4" visible="no" active="no"/>
+<layer number="5" name="Route5" color="4" fill="4" visible="no" active="no"/>
+<layer number="6" name="Route6" color="1" fill="8" visible="no" active="no"/>
+<layer number="7" name="Route7" color="4" fill="8" visible="no" active="no"/>
+<layer number="8" name="Route8" color="1" fill="2" visible="no" active="no"/>
+<layer number="9" name="Route9" color="4" fill="2" visible="no" active="no"/>
+<layer number="10" name="Route10" color="1" fill="7" visible="no" active="no"/>
+<layer number="11" name="Route11" color="4" fill="7" visible="no" active="no"/>
+<layer number="12" name="Route12" color="1" fill="5" visible="no" active="no"/>
+<layer number="13" name="Route13" color="4" fill="5" visible="no" active="no"/>
+<layer number="14" name="Route14" color="1" fill="6" visible="no" active="no"/>
+<layer number="15" name="Route15" color="4" fill="6" visible="no" active="no"/>
 <layer number="16" name="Bottom" color="1" fill="1" visible="no" active="no"/>
 <layer number="17" name="Pads" color="2" fill="1" visible="no" active="no"/>
@@
 <part name="R6" library="resistor" deviceset="R-US_" device="0204/7" value="47K"/>
 <part name="R7" library="resistor" deviceset="R-US_" device="0204/7" value="3.3K"/>
-<part name="R8" library="resistor" deviceset="R-US_" device="0204/7" value="1530"/>
 <part name="R9" library="resistor" deviceset="R-US_" device="0204/7" value="10"/>
 <part name="D1" library="diode" deviceset="1N4148" device="DO35-7"/>
@@
 <part name="J1" library="con-amp" deviceset="MTA03-100" device="" value="ZYX"/>
 <part name="J2" library="con-amp" deviceset="MTA02-100" device="" value="E-,E+"/>
+<part name="R8" library="resistor" deviceset="R-TRIMM" device="3296Y"/>
 </parts>
 <sheets>
@@
 <instance part="R6" gate="G$1" x="71.12" y="33.02" rot="R90"/>
 <instance part="R7" gate="G$1" x="71.12" y="5.08" rot="R90"/>
-<instance part="R8" gate="G$1" x="45.72" y="78.74"/>
 <instance part="R9" gate="G$1" x="-5.08" y="38.1" rot="R90"/>
 <instance part="D1" gate="G$1" x="78.74" y="17.78"/>
@@
 <instance part="J1" gate="G$1" x="33.02" y="96.52"/>
 <instance part="J2" gate="G$1" x="71.12" y="93.98"/>
+<instance part="R8" gate="G$1" x="43.18" y="78.74" rot="R90"/>
 </instances>
 <busses>
@@
 <pinref part="R2" gate="G$1" pin="2"/>
 <wire x1="142.24" y1="71.12" x2="142.24" y2="78.74" width="0.1524" layer="91"/>
-<pinref part="R8" gate="G$1" pin="2"/>
 <wire x1="142.24" y1="78.74" x2="109.22" y2="78.74" width="0.1524" layer="91"/>
+<wire x1="48.26" y1="78.74" x2="50.8" y2="78.74" width="0.1524" layer="91"/>
 <wire x1="50.8" y1="78.74" x2="55.88" y2="78.74" width="0.1524" layer="91"/>
 <wire x1="55.88" y1="78.74" x2="83.82" y2="78.74" width="0.1524" layer="91"/>
@@
 <wire x1="35.56" y1="93.98" x2="55.88" y2="93.98" width="0.1524" layer="91"/>
 <wire x1="55.88" y1="93.98" x2="55.88" y2="78.74" width="0.1524" layer="91"/>
+<pinref part="R8" gate="G$1" pin="E"/>
+<wire x1="50.8" y1="78.74" x2="50.8" y2="83.82" width="0.1524" layer="91"/>
+<pinref part="R8" gate="G$1" pin="S"/>
+<wire x1="50.8" y1="83.82" x2="43.18" y2="83.82" width="0.1524" layer="91"/>
 </segment>
 </net>
@@
 <pinref part="C2" gate="G$1" pin="1"/>
 <wire x1="33.02" y1="38.1" x2="33.02" y2="78.74" width="0.1524" layer="91"/>
-<pinref part="R8" gate="G$1" pin="1"/>
 <pinref part="L1" gate="G$1" pin="2"/>
-<wire x1="40.64" y1="78.74" x2="33.02" y2="78.74" width="0.1524" layer="91"/>
 <pinref part="J1" gate="G$1" pin="2"/>
+<wire x1="38.1" y1="78.74" x2="33.02" y2="78.74" width="0.1524" layer="91"/>
 <wire x1="33.02" y1="78.74" x2="20.32" y2="78.74" width="0.1524" layer="91"/>
 <wire x1="33.02" y1="93.98" x2="33.02" y2="78.74" width="0.1524" layer="91"/>
-</segment>
-</net>
+<pinref part="R8" gate="G$1" pin="A"/>
+</segment>
+</net>
